Commit message: - Change inverted_pendulum urdf to wippy - Update package name in urdf to urdfs - Use rviz config file in launch file

File: src/urdfs/urdf/wippy.urdf (robot description, URDF)
Before this commit: robot inverted_pendulum, 5 links, 4 joints
Links:
- link axle: geometry visual mesh filename=package://urdfs/meshes/axle.stl scale=1 1 1
- link chassis: geometry visual mesh filename=package://urdfs/meshes/chassis.stl scale=1 1 1
- link weight: geometry visual mesh filename=package://urdfs/meshes/weight.stl scale=1 1 1
- link wheel_left: geometry visual mesh filename=package://urdfs/meshes/wheel.stl scale=1 1 1
- link wheel_right: geometry visual mesh filename=package://urdfs/meshes/wheel.stl scale=1 1 1
